Commit message: XAdding new Files

File: my_package/description/robot.urdf.xacro (robot description, xacro)
@@ -2,3 +2,5 @@
 <robot xmlns:xacro="http://www.ros.org/wiki/xacro" name="robot">
    <xacro:include filename="robot_core.xacro"/>
+   <xacro:include filename="gazebo_control.xacro"/>
+   <xacro:include filename="lidar.xacro"/>
 </robot>

File: my_package/description/robot_core.xacro (robot description, xacro)
@@ -1,4 +1,12 @@
 <?xml version="1.0"?>
 <robot xmlns:xacro="http://www.ros.org/wiki/xacro">
+    <!-- Body dimensions -->
+    <xacro:property name="body_x" value="0.381"/>
+    <xacro:property name="body_y" value="0.191"/>
+    <xacro:property name="body_z" value="0.09242"/>
+    <!-- Wheel dim -->
+    <xacro:property name="wheel_radius" value="0.04918"/>
+    <xacro:property name="wheel_length" value="0.03935"/>
+    <xacro:property name="wheel_z"  value="-0.01492"/>
     <xacro:include filename="inertial_macros.xacro"/>
     <material name="white">
@@ -44,4 +52,7 @@
         </xacro:inertial_box>
     </link>
+    <gazebo reference="chassis">
+        <material>Gazebo/White</material>
+    </gazebo>
     <!-- Left Front Wheel -->
     <joint name="left_front_wheel_joint" type="continuous">
@@ -50,4 +61,6 @@
         <origin xyz="0.09525 0.111 0" rpy="-${pi/2} 0 0"/>
         <axis xyz="0 0 1"/>
+        <limit effort="1000" velocity="1000"/>
+        <dynamics damping="1.0" friction="1.0"/>
     </joint>
     <link name="left_front_wheel">
@@ -67,4 +80,7 @@
         </xacro:inertial_cylinder>
     </link>
+    <gazebo reference="left_front_wheel">
+        <material>Gazebo/Blue</material>
+    </gazebo>
     <!-- Right Front Wheel -->
     <joint name="right_front_wheel_joint" type="continuous">
@@ -73,4 +89,6 @@
         <origin xyz="0.09525 -0.111 0" rpy="${pi/2} 0 0"/>
         <axis xyz="0 0 -1"/>
+        <limit effort="1000" velocity="1000"/>
+        <dynamics damping="1.0" friction="1.0"/>
     </joint>
     <link name="right_front_wheel">
@@ -90,4 +108,7 @@
         </xacro:inertial_cylinder>
     </link>
+    <gazebo reference="right_front_wheel">
+        <material>Gazebo/Blue</material>
+    </gazebo>
     <!-- Left Back Wheel -->
     <joint name="left_back_wheel_joint" type="continuous">
@@ -96,4 +117,6 @@
         <origin xyz="-0.09525 0.111 0" rpy="-${pi/2} 0 0"/>
         <axis xyz="0 0 1"/>
+        <limit effort="1000" velocity="1000"/>
+        <dynamics damping="1.0" friction="1.0"/>
     </joint>
     <link name="left_back_wheel">
@@ -113,4 +136,7 @@
         </xacro:inertial_cylinder>
     </link>
+    <gazebo reference="left_back_wheel">
+        <material>Gazebo/Blue</material>
+    </gazebo>
     <!-- Right back Wheel -->
     <joint name="right_back_wheel_joint" type="continuous">
@@ -119,4 +145,6 @@
         <origin xyz="-0.09525 -0.111 0" rpy="${pi/2} 0 0"/>
         <axis xyz="0 0 -1"/>
+        <limit effort="1000" velocity="1000"/>
+        <dynamics damping="1.0" friction="1.0"/>
     </joint>
     <link name="right_back_wheel">
@@ -136,3 +164,6 @@
         </xacro:inertial_cylinder>
     </link>
+    <gazebo reference="right_back_wheel">
+        <material>Gazebo/Blue</material>
+    </gazebo>
 </robot>
